File: hellen-112-17.kicad_sch (KiCad schematic)
At the start: 1 part

Commit message: #3 #4 #5 #6
Parts:
- removed J?: rusefi_2x56_pin_conn, kicad6-libraries:rusefi_2x56_pin_connector, symbol rusefi_2x56_pin_connector:rusefi_2x56_pin_conn
- added C22: 470uF, Capacitor_SMD:CP_Elec_10x10.5, symbol Device:C_Polarized
- added F6 (x3): 12H1500D, hellen-one-common:PAD-1206-PAD, symbol hellen-one-common:Fuse-Pad-Pad
- added J1: rusefi_2x56_pin_conn, rusefi_2x56_pin_connector:rusefi_2x56_pin_connector, symbol rusefi_2x56_pin_connector:rusefi_2x56_pin_conn
- added M1: Module:mega_mcu100/0.1, hellen-one-mega-mcu100-0.1:mega-mcu100, symbol hellen-one-mega-mcu100-0.1:root_0_Mod-Hellen-MEGA_MCU100
- added M2: Module-power_12and5V-0.2, hellen-one-power_12and5V-0.2:power_12and5V, symbol hellen-one-power_12and5V:Module-power_12and5V-0.2
- added P6 (x13): Pad, hellen-one-common:PAD-TH, symbol hellen-one-common:Pad
- added Q? (x4): ISL9V3040D3S, Package_TO_SOT_SMD:TO-252-2, symbol Device:Q_NIGBT_GCE
- added R13, R14: Jumper-Pad-Pad, hellen-one-common:PAD-0805-PAD, symbol hellen-one-common:Jumper-Pad-Pad
- added R? (x4): DNP, Resistor_SMD:R_2512_6332Metric, symbol hellen-one-common:Res
- added R? (x4): 100k, hellen-one-common:R0603, symbol hellen-one-common:Res
- added R? (x4): 22, hellen-one-common:R0603, symbol hellen-one-common:Res
Connections:
- new net: Q?.1 (G), R?.1 (x4)
- new net: F6.1, J1.A56
- new net: J1.B52, R14.1
- new net: J1.B51, R13.1
- new net: F6.1, J1.A16
- new net: J1.B8, P6.1 (Pin_1)
- new net: J1.A8, P6.1 (Pin_1)
- new net: F6.1, J1.A55
- new net +12V: M2.E2 (V12)
- new net +12VA: F6.2, F6.2
- new net +12V_ETB: C22.1
- new net +12V_RAW: M2.V1 (V12_PERM), M2.V3 (V12_RAW)
- new net +3V3: J1.A26
- new net +5V: M2.E4 (V5)
- new net +5VP: J1.A25, J1.B10, M2.V4 (5VP)
- new net 101_out: J1.A1
- new net 102_out: J1.A2
- new net 107: J1.A7, P6.1 (Pin_1)
- new net ANALOG_MAF: J1.B33
- new net ANALOG_SUPPLY_MAP: J1.B23
- new net ANALOG_TPS: J1.A38
- new net A/C_PRESSURE: J1.A19, P6.1 (Pin_1)
- new net CAM: J1.B31
- new net CAN+: J1.A32, M1.W11 (CANH)
- new net CAN-: J1.A44, M1.W12 (CANL)
- new net CLT: J1.B15
- new net COIL1 output: J1.B56, Q?.2 (C), R?.2
- new net COIL2 output: J1.B53, Q?.2 (C), R?.2
- new net COIL3 output: J1.B54, Q?.2 (C), R?.2
- new net COIL4 output: J1.B55, Q?.2 (C), R?.2
- new net CRANK_VR+: J1.B13
- new net CRANK_VR-: J1.B1
- new net ENGINE_RADIATOR_FAN: J1.A41
- new net ETB+: R13.2
- new net ETB-: R14.2
- new net ETB_PWM: M1.E17 (OUT_INJ1_(PD3))
- new net FUEL_LVL: J1.A12
- new net FUEL_PUMP_RELAY: J1.A42
- new net GND: J1.A53, J1.A54, M1.G (GND)
- new net GNDA_A3: J1.A3, P6.1 (Pin_1)
- new net GND_A4: J1.A4, P6.1 (Pin_1)
- new net GND_A5: J1.A5, P6.1 (Pin_1)
- new net GND_A6: J1.A6
- new net GND_B4: J1.B4, P6.1 (Pin_1)
- new net GND_B47: J1.B47
- new net GND_B5: J1.B5, P6.1 (Pin_1)
- new net GND_B50: C22.2, J1.B50, M2.S1 (GND), Q?.3 (E), Q?.3 (E), Q?.3 (E), Q?.3 (E), R?.1, R?.1, R?.1, R?.1
- new net GND_B6: J1.B6, P6.1 (Pin_1)
- new net GND_B7: J1.B7, P6.1 (Pin_1)
- new net IAT: J1.B27
- new net IGN1: M1.W10 (IGN1_(PC13)), R?.1, R?.2, R?.2
- new net IGN2: M1.W9 (IGN2_(PE5)), R?.1, R?.2, R?.2
- new net IGN3: M1.W8 (IGN3_(PE4)), R?.1, R?.2, R?.2
- new net IGN4: M1.W7 (IGN4_(PE3)), R?.1, R?.2, R?.2
- new net INJ1: J1.B44
- new net INJ2: J1.B42
- new net INJ3: J1.B43
- new net INJ4: J1.B45
- new net IN_A23: J1.A23
- new net IN_ANALOG: J1.A11
- new net IN_BRAKE: J1.A13
- new net IN_VIGN: M2.V2 (IN_VIGN)
- new net IN_VSS: J1.B32
- new net K-LINE: J1.A27
- new net KNOCK1: J1.B37
- new net KNOCK2: J1.B38
- new net MAIN_RELAY_CNTRL: J1.A15
- new net MAP: J1.B19
- new net OUT_FUEL: J1.A29
- new net OUT_LOW_SIDE: J1.B46
- new net OUT_RELAY_A20: J1.A20
- new net OUT_RELAY_A40: J1.A40
- new net OUT_RELAY_A51: J1.A51
- new net OUT_RELAY_A52: J1.A52
- new net OUT_TACH: J1.A28
- new net PEDAL_POSITION1: J1.A21
- new net PEDAL_POSITION2: J1.A14
- new net PWR_EN: M1.N20 (OUT_PWR_EN_(PE10)), M2.E5 (EN_5VP)
- new net SWITCH_A34: J1.A34
- new net SWITCH_A35: J1.A35
- new net SWITCH_A36: J1.A36
- new net SWITCH_A47: J1.A47
- new net THROTTLE_POSITION_1: J1.B3
- new net THROTTLE_POSITION_2: J1.B20
- new net TLS115_PG: M2.E6 (PG_5VP)
- new net VBAT: M1.N17 (VBAT), M2.E1 (VBAT)
- new net VIGN: M1.E5 (IN_VIGN_(PA5)), M2.E3 (VIGN)
- new net VOLTAGE_FROM_KEY: F6.2
- new net Сonditioner_relay: J1.A31
- no-connect marks 0 -> 40
Other:
- added sheet ETB (DC_MOTOR_0.1.kicad_sch)
- note added: "Optional"
- note added: "TLE9201 motor driver"
- title: hellen-112-17 -> adapter-board-me17-112

Commit message: пронумеровала, перенесла изменения на плату
Parts:
- removed P6 (x2): Pad, hellen-one-common:PAD-TH, symbol hellen-one-common:Pad
Connections:
- net ETB_PWM: now also M1.E18 (OUT_PWM1_(PD13)); no longer M1.E17 (OUT_INJ1_(PD3))
- net lowside_quad/IN4: now reaches M1.E14 (OUT_INJ4_(PD10))
- net lowside_quad/IN2: now reaches M1.E15 (OUT_INJ3_(PD11))
- net lowside_quad/IN3: now reaches M1.E16 (OUT_INJ2_(PA9))
- new net lowside_quad/IN1: M1.E17 (OUT_INJ1_(PD3))
Other:
- added sheet lowside_quad (lowside_quad.kicad_sch)

Commit message: Upd SCH
Parts:
- removed C22: 470uF, Capacitor_SMD:CP_Elec_10x10.5, symbol Device:C_Polarized
- removed unit 3 of J1
- removed unit 4 of J1
- removed unit 2 of J1
- removed P6 (x11): Pad, hellen-one-common:PAD-TH, symbol hellen-one-common:Pad
- removed Q? (x4): ISL9V3040D3S, Package_TO_SOT_SMD:TO-252-2, symbol Device:Q_NIGBT_GCE
- removed R? (x4): DNP, Resistor_SMD:R_2512_6332Metric, symbol hellen-one-common:Res
- removed R? (x4): 100k, hellen-one-common:R0603, symbol hellen-one-common:Res
- removed R? (x4): 22, hellen-one-common:R0603, symbol hellen-one-common:Res
- added G1, G2: PROTO_AREA, hellen-one-common:PROTO_AREA, symbol hellen-one-common:PROTO_AREA
- added J1: USB_B_Mini, hellen-one-common:USB-MINI-B-VERTICAL, symbol hellen-one-common:USB_B_Mini
- added M2: Module-vr-max9924-0.1, hellen-one-vr-max9924-0.1:vr-max9924, symbol vr-max9924:Module-vr-max9924-0.1
- added M3: Module-knock-0.2, hellen-one-knock-0.2:knock, symbol hellen-one-knock-0.2:Module-knock-0.2
- added M5: Module-lin-0.1, hellen-one-lin-0.1:lin, symbol hellen-one-lin-0.1:Module-lin-0.1
- added R1, R10, R11, R12, R15, R16, R2, R3, R4, R5, R6, R7, R8, R9: Jumper-Pad-Pad, hellen-one-common:PAD-0805-PAD, symbol hellen-one-common:Jumper-Pad-Pad
- added R92: 4.7k, hellen-one-common:R0603, symbol hellen-one-common:Res
- J1: footprint rusefi_2x56_pin_connector:rusefi_2x56_pin_connector -> kicad6-libraries:rusefi_2x56_pin_connector
- renumbered M2 to M1, M1 to M4
Connections:
- net +12VA is gone; now on net +12V_RAW: F6.2, F6.2
- net ETB- is gone; now on net GNDA: R14.2
- net GND_B50 is gone; now on net GND: M1.S1 (GND)
- net VOLTAGE_FROM_KEY is gone; now on net IN_VIGN: F6.2
- net lowside_quad/IN1 is gone; now on net INJ1: M4.E17 (OUT_INJ1_(PD3))
- net lowside_quad/IN2 is gone; now on net INJ3: M4.E15 (OUT_INJ3_(PD11))
- net lowside_quad/IN3 is gone; now on net INJ2: M4.E16 (OUT_INJ2_(PA9))
- net lowside_quad/IN4 is gone; now on net INJ4: M4.E14 (OUT_INJ4_(PD10))
- net +12V: now also M5.N1 (12V), M5.V1 (12V)
- net +12V_RAW: now also G1.10, G1.15, G1.5
- net +3.3V: now also M4.N21 (V33)
- net +3V3: now also R92.1; no longer J1.A26
- net +5V: now also M4.N22 (VCC)
- net +5VP: now also J1.37, J1.66, R11.2, R6.2, R7.2, R8.2; no longer J1.A25
- net CAN+: now also J1.32
- net CAN-: now also J1.44
- net ETB_DIR: now also M4.E8 (SPI2_MISO_(PB14))
- net ETB_DIS: now also M4.E9 (SPI2_MOSI_(PB15))
- net ETB_PWM: now also M4.E23 (OUT_PWM6_(PD14)); no longer M4.E18 (OUT_PWM1_(PD13))
- net GND: now also J1.106, J1.53, J1.54, G1.1, G1.11, G1.12, G1.2, G1.6, G1.7, J1.5 (GND), J1.6 (Shield), M2.G (GND), M3.E2 (GND), M5.E1 (GND), M5.S1 (GND), R2.2
- net IN_VSS: now also J1.88, M4.S3 (IN_D2_(PE13))
- net OUT_FUEL: now also J1.29
- net OUT_TACH: now also J1.28; no longer J1.A28
- net TLS115_PG: now also M4.N12 (SPI3_MOSI_(PC12))
- net at F6.1: now also J1.56
- net at R14.1: now also J1.94
- net at R13.1: now also J1.93
- net at F6.1: now also J1.16; no longer J1.A16
- net +5VA: now reaches M4.E1 (V5A_SWITCHABLE)
- net +5VA: now also M4.W2 (V5A_SWITCHABLE), G1.14, G1.4, G1.9, M2.E4 (V5_IN), M3.E1 (V5A), M5.V3 (5V)
- net lowside_quad1/IN4: now reaches M4.E10 (OUT_INJ8_(PD12))
- net lowside_quad1/IN2: now reaches M4.E11 (OUT_INJ7_(PD15))
- net lowside_quad1/IN3: now reaches M4.E12 (OUT_INJ6_(PA8))
- net lowside_quad1/IN1: now reaches M4.E13 (OUT_INJ5_(PD2))
- net lowside_weak/IN6: now reaches M4.E19 (OUT_PWM2_(PC6))
- net lowside_weak/IN7: now reaches M4.E20 (OUT_PWM3_(PC7))
- net lowside_weak/IN8: now reaches M4.E21 (OUT_PWM4_(PC8))
- net lowside_weak/IN9: now reaches M4.E22 (OUT_PWM5_(PC9))
- net IN_DIGITAL_147_HS: now reaches M4.E6 (SPI2_CS_/_CAN2_RX_(PB12))
- net IN_DIGITAL_147_HS: now also J1.47
- net IN_DIGITAL_123: now reaches M4.E7 (SPI2_SCK_/_CAN2_TX_(PB13))
- net IN_DIGITAL_123: now also J1.23
- net VBUS: now reaches M4.N1 (VBUS)
- net VBUS: now also J1.1 (VBUS)
- net IN_DIGITAL_134_HS: now reaches M4.N10 (SPI3_SCK_(PC10))
- net IN_DIGITAL_134_HS: now also J1.34
- net IN_DIGITAL_135_HS: now reaches M4.N11 (SPI3_MISO_(PC11))
- net IN_DIGITAL_135_HS: now also J1.35
- net +3.3VA: now reaches M4.N15 (V33_SWITCHABLE)
- net +3.3VA: now also G1.13, G1.3, G1.8
- net at M4.N18 (UART8_RX_(PE0)): now also M5.V2 (UART_RX), R92.2
- net at M4.N19 (UART8_TX_(PE1)): now also M5.V5 (UART_TX)
- net USB-: now reaches M4.N2 (USBM_(PA11))
- net USB-: now also J1.2 (D-)
- net USB+: now reaches M4.N3 (USBP_(PA12))
- net USB+: now also J1.3 (D+)
- net IN_DIGITAL_136_HS: now reaches M4.N9 (SPI3_CS_(PA15))
- net IN_DIGITAL_136_HS: now also J1.36
- net IN_DIGITAL_120: now reaches M4.S1 (IN_D4_(PE15))
- net IN_DIGITAL_120: now also J1.20
- net IN_PPS2: now reaches M4.S10 (IN_O2S2_(PA1))
- net IN_PPS2: now also R4.2
- net IN_TPS2: now reaches M4.S11 (IN_O2S_/_CAN_WAKEUP_(PA0))
- net IN_TPS2: now also J1.76
- net IN_AV_109: now reaches M4.S12 (IN_MAP2_(PC1))
- net IN_AV_109: now also J1.9
- net IN_MAP: now reaches M4.S13 (IN_MAP1_(PC0))
- net IN_MAP: now also J1.75
- net CRANK_VR: now reaches M4.S14 (IN_CRANK_(PB1))
- net CRANK_VR: now also M2.E3 (OUT)
- net IN_KNOCK: now reaches M4.S15 (IN_KNOCK_(PA2))
- net IN_KNOCK: now also M3.E3 (OUT_KNOCK)
- net IN_AV_107: now reaches M4.S16 (IN_CAM_(PA6))
- net IN_AV_107: now also R1.2
- net MAF_DIGITAL: now reaches M4.S17 (IN_VSS_(PE11))
- net IN_TPS1: now reaches M4.S18 (IN_TPS_(PA4))
- net IN_TPS1: now also J1.59
- net IN_PPS1: now reaches M4.S19 (IN_PPS_(PA3))
- net IN_PPS1: now also R5.2
- net IN_DIGITAL_113: now reaches M4.S2 (IN_D3_(PE14))
- net IN_DIGITAL_113: now also J1.13
- net IN_IAT: now reaches M4.S20 (IN_IAT_(PC3))
- net IN_IAT: now also J1.83
- net IN_CLT: now reaches M4.S21 (IN_CLT_(PC2))
- net IN_CLT: now also J1.71
- net IN_CAM: now reaches M4.S4 (IN_D1_(PE12))
- net IN_CAM: now also J1.87
- net VREF2: now reaches M4.S5 (VREF2)
- net VREF2: now also M3.W2 (VREF)
- net IN_AV_119: now reaches M4.S6 (IN_AUX4_(PA7))
- net IN_AV_119: now also J1.19
- net IN_AV_112: now reaches M4.S7 (IN_AUX3_(PC5))
- net IN_AV_112: now also J1.12
- net IN_AV_111: now reaches M4.S8 (IN_AUX2_(PC4/PE9))
- net IN_AV_111: now also R3.2
- net IN_AV_110: now reaches M4.S9 (IN_AUX1_(PB0))
- net IN_AV_110: now also J1.10
- net GNDA: now reaches M4.W1 (GNDA)
- net GNDA: now also J1.103, J1.3, J1.4, J1.5, J1.6, J1.60, J1.61, J1.62, J1.63, J1.64
- net lowside_weak/IN4: now reaches M4.W3 (IGN8_(PE6))
- net lowside_weak/IN3: now reaches M4.W4 (IGN7_(PB9))
- net lowside_weak/IN2: now reaches M4.W5 (IGN6_(PB8))
- net lowside_weak/IN1: now reaches M4.W6 (IGN5_(PE2))
- net at F6.1: now also J1.55
- removed net 101_out: J1.A1
- removed net 102_out: J1.A2
- removed net 107: J1.A7
- removed net A/C_PRESSURE: J1.A19
- net ETB+ renamed IN_KNOCK_RAW
- net IN_KNOCK_RAW: now also M3.W1 (IN_KNOCK)
- removed net FUEL_LVL: J1.A12
- removed net GNDA_A3: J1.A3
- removed net GND_A4: J1.A4
- removed net GND_A5: J1.A5
- removed net GND_A6: J1.A6
- removed net IN_A23: J1.A23
- removed net IN_ANALOG: J1.A11
- removed net IN_BRAKE: J1.A13
- removed net K-LINE: J1.A27
- removed net MAIN_RELAY_CNTRL: J1.A15
- removed net OUT_RELAY_A20: J1.A20
- removed net PEDAL_POSITION1: J1.A21
- removed net PEDAL_POSITION2: J1.A14
- new net: J1.38, R8.1
- new net: G2.1, G2.11, G2.6
- new net: G2.10, G2.15, G2.5
- new net: G2.12, G2.2, G2.7
- new net: G2.13, G2.3, G2.8
- new net: G2.14, G2.4, G2.9
- new net: J1.69, R10.1
- new net: J1.14, R4.1
- new net: J1.57, R9.1
- new net: J1.89, R12.1
- new net: J1.11, R3.1
- new net: J1.79, R11.1
- new net: J1.8, R2.1
- new net: J1.25, R6.1
- new net: J1.21, R5.1
- new net: J1.107, R15.1
- new net: J1.26, R7.1
- new net: J1.7, R1.1
- new net: J1.108, R16.1
- new net IN_CRANK_VR+: M2.W2 (VR+), R10.2
- new net IN_CRANK_VR-: M2.W1 (VR-), R9.2
- new net IN_MAF_DIGITAL: R12.2
- new net K-Line: J1.27, M5.V4 (LIN)
- new net OUT_AC: J1.31
- new net OUT_ETB+: R15.2
- new net OUT_ETB-: R16.2
- new net OUT_FAN_RELAY: J1.41
- new net OUT_FUEL_PUMP_RELAY: J1.42
- new net OUT_IGN1: J1.112
- new net OUT_IGN2: J1.109
- new net OUT_IGN3: J1.110
- new net OUT_IGN4: J1.111
- new net OUT_INJ1: J1.100
- new net OUT_INJ2: J1.98
- new net OUT_INJ3: J1.99
- new net OUT_INJ4: J1.101
- new net OUT_LS_101: J1.1
- new net OUT_LS_102: J1.2
- new net OUT_LS_235: J1.91
- new net OUT_LS_246: J1.102
- new net OUT_MAIN_RELAY: J1.15
- new net OUT_RELAY_140: J1.40
- new net OUT_RELAY_151: J1.51
- new net OUT_RELAY_152: J1.52
- new net lowside_weak/IN5: M4.E18 (OUT_PWM1_(PD13))
- no-connect marks 40 -> 54
Other:
- added sheet FREQ_DIVIDER (FREQ_DIVIDER.kicad_sch)
- added sheet IGN_QUAD (ign_quad.kicad_sch)
- added sheet lowside_quad1 (lowside_quad.kicad_sch)
- added sheet lowside_weak (LS_weak.kicad_sch)
- note added: "12V PU"
- note added: "TODO: ign serier resistor 33"
- note removed: "Optional"
- company: rusEFI -> rusEFI.com
- title: adapter-board-me17-112 -> hellen-112-17
- moved on the sheet: F6, M1, M4

Commit message: Export
Parts:
- added G3: LOGO, hellen-one-common:LOGO, symbol hellen-one-common:LOGO
- added G4: RUSEFI_LOGO, kicad6-libraries:rusefi_logo, symbol rusefi_logo:RUSEFI_LOGO
- added R30 (x2): 4.7k, hellen-one-common:R0603, symbol hellen-one-common:Res
Connections:
- net +3V3 is gone; now on net +3.3V: R92.1
- net +12V: now also R30.2, R30.2
- net IN_DIGITAL_123: no longer M4.E7 (SPI2_SCK_/_CAN2_TX_(PB13))
- net IN_DIGITAL_134_HS: no longer M4.N10 (SPI3_SCK_(PC10))
- net IN_DIGITAL_135_HS: no longer M4.N11 (SPI3_MISO_(PC11))
- net IN_DIGITAL_136_HS: no longer M4.N9 (SPI3_CS_(PA15))
- net IN_DIGITAL_147_HS: no longer M4.E6 (SPI2_CS_/_CAN2_RX_(PB12))
- net OUT_FUEL: now also R30.1
- net OUT_TACH: now also R30.1
- net TLS115_PG: now also M4.N9 (SPI3_CS_(PA15)); no longer M1.E6 (PG_5VP), M4.N12 (SPI3_MOSI_(PC12))
- net IN_CRANK+: now reaches J1.69, R10.1
- net IN_CRANK-: now reaches J1.57, R9.1
- new net DIGITAL_123: M4.N12 (SPI3_MOSI_(PC12))
- new net DIGITAL_134_HS: M4.E7 (SPI2_SCK_/_CAN2_TX_(PB13))
- new net DIGITAL_135_HS: M4.E6 (SPI2_CS_/_CAN2_RX_(PB12))
- new net DIGITAL_136_HS: M4.N10 (SPI3_SCK_(PC10))
- new net DIGITAL_147_HS: M4.N11 (SPI3_MISO_(PC11))
- new net IN_TLS115_PG: M1.E6 (PG_5VP)
Other:
- added sheet dinput6 (dinput6.kicad_sch)
- note added: "Analog inputs (sensors)"
- note added: "Bus types"
- note added: "DC Motor"
- note added: "Discrete inputs"
- note added: "General purpose bus"
- note added: "Ignition"
- note added: "Injection"
- note added: "LS & HS outputs"
- note removed: "12V PU"
- moved on the sheet: F6, J1, M2, M3, R10, R9

Commit message: Update mm100, connector, replace
Parts:
- removed M4: Module:mega_mcu100/0.1, hellen-one-mega-mcu100-0.1:mega-mcu100, symbol hellen-one-mega-mcu100-0.1:root_0_Mod-Hellen-MEGA_MCU100
- added M4: Module:mega-mcu100/0.1, hellen-one-mega-mcu100-0.1:mega-mcu100, symbol hellen-one-mega-mcu100-0.1:Module{colon}mega-mcu100/0.1
Connections:
- net +3.3V: now also M4.N21 (V33)
- net +3.3VA: now also M4.N15 (V33_SWITCHABLE)
- net +5V: now also M4.N22 (VCC)
- net +5VA: now also M4.E1 (V5A_SWITCHABLE), M4.W2 (V5A_SWITCHABLE)
- net CAN+: now also M4.W11 (CANH)
- net CAN-: now also M4.W12 (CANL)
- net CRANK_VR: now also M4.S14 (IN_CRANK_(PB1))
- net DIGITAL_123: now also M4.N12 (SPI3_MOSI_(PC12))
- net DIGITAL_134_HS: now also M4.E7 (SPI2_SCK_/_CAN2_TX_(PB13))
- net DIGITAL_135_HS: now also M4.E6 (SPI2_CS_/_CAN2_RX_(PB12))
- net DIGITAL_136_HS: now also M4.N10 (SPI3_SCK_(PC10))
- net DIGITAL_147_HS: now also M4.N11 (SPI3_MISO_(PC11))
- net ETB_DIR: now also M4.E8 (SPI2_MISO_(PB14))
- net ETB_DIS: now also M4.E9 (SPI2_MOSI_(PB15))
- net ETB_PWM: now also M4.E23 (OUT_PWM6_(PD14))
- net GND: now also M4.G (GND)
- net GNDA: now also M4.W1 (GNDA)
- net IGN1: now also M4.W10 (IGN1_(PC13))
- net IGN2: now also M4.W9 (IGN2_(PE5))
- net IGN3: now also M4.W8 (IGN3_(PE4))
- net IGN4: now also M4.W7 (IGN4_(PE3))
- net INJ1: now also M4.E17 (OUT_INJ1_(PD3))
- net INJ2: now also M4.E16 (OUT_INJ2_(PA9))
- net INJ3: now also M4.E15 (OUT_INJ3_(PD11))
- net INJ4: now also M4.E14 (OUT_INJ4_(PD10))
- net IN_AV_107: now also M4.S16 (IN_CAM_(PA6))
- net IN_AV_109: now also M4.S12 (IN_MAP2_(PC1))
- net IN_AV_110: now also M4.S9 (IN_AUX1_(PB0))
- net IN_AV_111: now also M4.S8 (IN_AUX2_(PC4/PE9))
- net IN_AV_112: now also M4.S7 (IN_AUX3_(PC5))
- net IN_AV_119: now also M4.S6 (IN_AUX4_(PA7))
- net IN_CAM: now also M4.S4 (IN_D1_(PE12))
- net IN_CLT: now also M4.S21 (IN_CLT_(PC2))
- net IN_DIGITAL_113: now also M4.S2 (IN_D3_(PE14))
- net IN_DIGITAL_120: now also M4.S1 (IN_D4_(PE15))
- net IN_IAT: now also M4.S20 (IN_IAT_(PC3))
- net IN_KNOCK: now also M4.S15 (IN_KNOCK_(PA2))
- net IN_MAP: now also M4.S13 (IN_MAP1_(PC0))
- net IN_PPS1: now also M4.S19 (IN_PPS_(PA3))
- net IN_PPS2: now also M4.S10 (IN_O2S2_(PA1))
- net IN_TPS1: now also M4.S18 (IN_TPS_(PA4))
- net IN_TPS2: now also M4.S11 (IN_O2S_/_CAN_WAKEUP_(PA0))
- net IN_VSS: now also M4.S3 (IN_D2_(PE13))
- net MAF_DIGITAL: now also M4.S17 (IN_VSS_(PE11))
- net PWR_EN: now also M4.N20 (OUT_PWR_EN_(PE10))
- net TLS115_PG: now also M4.N9 (SPI3_CS_(PA15))
- net USB+: now also M4.N3 (USBP_(PA12))
- net USB-: now also M4.N2 (USBM_(PA11))
- net VBAT: now also M4.N17 (VBAT)
- net VBUS: now also M4.N1 (VBUS)
- net VIGN: now also M4.E5 (IN_VIGN_(PA5))
- net VREF2: now also M4.S5 (VREF2)
- net at M5.V2 (UART_RX), R92.2: now also M4.N18 (UART8_RX_(PE0))
- net at M5.V5 (UART_TX): now also M4.N19 (UART8_TX_(PE1))
- new net AC: M4.E20 (OUT_PWM3_(PC7))
- new net FAN_RELAY: M4.E21 (OUT_PWM4_(PC8))
- new net FUEL: M4.E19 (OUT_PWM2_(PC6))
- new net FUEL_PUMP_RELAY: M4.E22 (OUT_PWM5_(PC9))
- new net LS_101: M4.E13 (OUT_INJ5_(PD2))
- new net LS_102: M4.E12 (OUT_INJ6_(PA8))
- new net LS_235: M4.E11 (OUT_INJ7_(PD15))
- new net LS_246: M4.E10 (OUT_INJ8_(PD12))
- new net MAIN_RELAY: M4.W3 (IGN8_(PE6))
- new net RELAY_140: M4.W4 (IGN7_(PB9))
- new net RELAY_151: M4.W6 (IGN5_(PE2))
- new net RELAY_152: M4.W5 (IGN6_(PB8))
- new net TACH: M4.E18 (OUT_PWM1_(PD13))
Other:
- note removed: "TODO: ign serier resistor 33"
- moved on the sheet: F6

Commit message: #18, #19
Parts:
- added R54: Jumper-Pad-Pad, hellen-one-common:PAD-0805-PAD, symbol hellen-one-common:Jumper-Pad-Pad
Connections:
- net +5VP: now also R54.2; no longer J1.37 (37A)
- net AC renamed AC_RELAY
- net FUEL renamed FUEL_CONSUMPTION
- net OUT_AC renamed OUT_AC_RELAY
- net OUT_FUEL renamed OUT_FUEL_CONSUMPTION
- new net: J1.37 (37A), R54.1
Changed lines of the file:
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@@
     (effects (font (size 1.27 1.27)) (justify left bottom))
   )
-  (label "TACH" (at 175.26 118.11 0) (fields_autoplaced)
+  (label "TACH" (at 166.37 118.11 0) (fields_autoplaced)
     (effects (font (size 1.27 1.27)) (justify left bottom))
   )
@@
     (effects (font (size 1.27 1.27)) (justify right bottom))
   )
-  (label "OUT_AC" (at 76.2 93.98 180) (fields_autoplaced)
+  (label "OUT_AC_RELAY" (at 76.2 93.98 180) (fields_autoplaced)
     (effects (font (size 1.27 1.27)) (justify right bottom))
   )
@@
     (effects (font (size 1.27 1.27)) (justify right bottom))
   )
-  (label "AC" (at 175.26 123.19 0) (fields_autoplaced)
+  (label "AC_RELAY" (at 166.37 123.19 0) (fields_autoplaced)
+    (effects (font (size 1.27 1.27)) (justify left bottom))
+  )
+  (label "OUT_FUEL_CONSUMPTION" (at 88.9 90.17 0) (fields_autoplaced)
     (effects (font (size 1.27 1.27)) (justify left bottom))
   )
@@
     (effects (font (size 1.27 1.27)) (justify right bottom))
   )
-  (label "OUT_FUEL" (at 88.9 90.17 0) (fields_autoplaced)
-    (effects (font (size 1.27 1.27)) (justify left bottom))
-  )
   (label "IN_CRANK_VR+" (at 76.2 195.58 180) (fields_autoplaced)
     (effects (font (size 1.27 1.27)) (justify right bottom))
@@
     (effects (font (size 1.27 1.27)) (justify left bottom))
   )
-  (label "OUT_AC" (at 88.9 92.71 0) (fields_autoplaced)
+  (label "OUT_AC_RELAY" (at 88.9 92.71 0) (fields_autoplaced)
     (effects (font (size 1.27 1.27)) (justify left bottom))
   )
@@
     (effects (font (size 1.27 1.27)) (justify left bottom))
   )
-  (label "FUEL_PUMP_RELAY" (at 175.26 128.27 0) (fields_autoplaced)
+  (label "FUEL_PUMP_RELAY" (at 166.37 128.27 0) (fields_autoplaced)
     (effects (font (size 1.27 1.27)) (justify left bottom))
   )
@@
     (effects (font (size 1.27 1.27)) (justify left bottom))
   )
+  (label "FUEL_CONSUMPTION" (at 166.37 120.65 0) (fields_autoplaced)
+    (effects (font (size 1.27 1.27)) (justify left bottom))
+  )
   (label "OUT_TACH" (at 88.9 87.63 0) (fields_autoplaced)
     (effects (font (size 1.27 1.27)) (justify left bottom))
@@
     (effects (font (size 1.27 1.27)) (justify right bottom))
   )
-  (label "OUT_FUEL" (at 76.2 88.9 180) (fields_autoplaced)
+  (label "OUT_FUEL_CONSUMPTION" (at 76.2 88.9 180) (fields_autoplaced)
     (effects (font (size 1.27 1.27)) (justify right bottom))
   )
@@
     (effects (font (size 1.27 1.27)) (justify right bottom))
   )
-  (label "FAN_RELAY" (at 175.26 125.73 0) (fields_autoplaced)
+  (label "FAN_RELAY" (at 166.37 125.73 0) (fields_autoplaced)
     (effects (font (size 1.27 1.27)) (justify left bottom))
   )
@@
   )
   (label "OUT_INJ4" (at 151.13 97.79 0) (fields_autoplaced)
-    (effects (font (size 1.27 1.27)) (justify left bottom))
-  )
-  (label "FUEL" (at 175.26 120.65 0) (fields_autoplaced)
     (effects (font (size 1.27 1.27)) (justify left bottom))
   )
@@
     )
   )
-  (symbol (lib_id "power:+5VP") (at 26.67 109.22 270) (unit 1)
-    (in_bom yes) (on_board yes) (dnp no)
-    (property "Reference" "#PWR?" (at 22.86 109.22 0)
-      (effects (font (size 1.27 1.27)) hide)
-    )
-    (property "Value" "+5VP" (at 31.75 109.22 90)
-      (effects (font (size 1.27 1.27)))
-    )
-    (property "Footprint" "" (at 26.67 109.22 0)
-      (effects (font (size 1.27 1.27)) hide)
-    )
-    (property "Datasheet" "" (at 26.67 109.22 0)
+  (symbol (lib_id "power:+5VP") (at 36.83 109.22 270) (unit 1)
+    (in_bom yes) (on_board yes) (dnp no)
+    (property "Reference" "#PWR?" (at 33.02 109.22 0)
+      (effects (font (size 1.27 1.27)) hide)
+    )
+    (property "Value" "+5VP" (at 41.91 109.22 90)
+      (effects (font (size 1.27 1.27)))
+    )
+    (property "Footprint" "" (at 36.83 109.22 0)
+      (effects (font (size 1.27 1.27)) hide)
+    )
+    (property "Datasheet" "" (at 36.83 109.22 0)
       (effects (font (size 1.27 1.27)) hide)
     )
@@
         )
       )
+    )
+  )
+  (symbol (lib_id "hellen-one-common:Jumper-Pad-Pad") (at 31.75 109.22 0) (unit 1)
+    (in_bom yes) (on_board yes) (dnp no)
+    (property "Reference" "R54" (at 36.3801 108.3891 0)
+      (effects (font (size 1.016 1.016)))
+    )
+    (property "Value" "Jumper-Pad-Pad" (at 31.75 110.998 0)
+      (effects (font (size 1.016 1.016)) hide)
+    )
+    (property "Footprint" "hellen-one-common:PAD-0805-PAD" (at 31.75 113.03 0)
+      (effects (font (size 1.524 1.524)) hide)
+    )
+    (property "Datasheet" "" (at 31.75 109.22 0)
+      (effects (font (size 1.524 1.524)) hide)
+    )
+    (property "LCSC" "C17477" (at 31.75 113.03 0)
+      (effects (font (size 1.27 1.27)) hide)
+    )
+    (pin "1")
+    (pin "2")
+    (instances
+      (project "hellen-112-17"
+        (path "/ac264c30-3e9a-4be2-b97a-9949b68bd497"
+          (reference "R54") (unit 1)
+        )
+      )
