File: hellen-112-17.kicad_sch (KiCad schematic)
At the start: 34 parts, among them J1 USB_B_Mini, J1 rusefi_2x56_pin_conn, M1 Module-power_12and5V-0.2, M2 Module-vr-max9924-0.1, M3 Module-knock-0.2, M4 Module:mega-mcu100/0.1, M5 Module-lin-0.1

Commit message: MM100_0.2
Parts:
- removed M4: Module:mega-mcu100/0.1, hellen-one-mega-mcu100-0.1:mega-mcu100, symbol hellen-one-mega-mcu100-0.1:Module{colon}mega-mcu100/0.1
- added M4: Module:mega-mcu100/0.2, hellen-one-mega-mcu100-0.2:mega-mcu100, symbol hellen-one-mega-mcu100-0.2:Module{colon}mega-mcu100/0.2
Connections:
- net +3.3V: now also M4.N21 (V33)
- net +3.3VA: now also M4.N15 (V33_SWITCHABLE)
- net +5V: now also M4.N22 (VCC)
- net +5VA: now also M4.E1 (V5A_SWITCHABLE), M4.W2 (V5A_SWITCHABLE)
- net AC_RELAY: now also M4.E20 (OUT_PWM3_(PC7))
- net CAN+: now also M4.W11 (CANH)
- net CAN-: now also M4.W12 (CANL)
- net CRANK_VR: now also M4.S14 (IN_CRANK_(PB1))
- net DIGITAL_123: now also M4.N12 (SPI3_MOSI_(PC12))
- net DIGITAL_134_HS: now also M4.E7 (SPI2_SCK_/_CAN2_TX_(PB13))
- net DIGITAL_135_HS: now also M4.E6 (SPI2_CS_/_CAN2_RX_(PB12))
- net DIGITAL_136_HS: now also M4.N10 (SPI3_SCK_(PC10))
- net DIGITAL_147_HS: now also M4.N11 (SPI3_MISO_(PC11))
- net ETB_DIR: now also M4.E8 (SPI2_MISO_(PB14))
- net ETB_DIS: now also M4.E9 (SPI2_MOSI_(PB15))
- net ETB_PWM: now also M4.E23 (OUT_PWM6_(PD14))
- net FAN_RELAY: now also M4.E21 (OUT_PWM4_(PC8))
- net FUEL_CONSUMPTION: now also M4.E19 (OUT_PWM2_(PC6))
- net FUEL_PUMP_RELAY: now also M4.E22 (OUT_PWM5_(PC9))
- net GND: now also M4.G (GND)
- net GNDA: now also M4.W1 (GNDA)
- net IGN1: now also M4.W10 (IGN1_(PC13))
- net IGN2: now also M4.W9 (IGN2_(PE5))
- net IGN3: now also M4.W8 (IGN3_(PE4))
- net IGN4: now also M4.W7 (IGN4_(PE3))
- net INJ1: now also M4.E17 (OUT_INJ1_(PD3))
- net INJ2: now also M4.E16 (OUT_INJ2_(PA9))
- net INJ3: now also M4.E15 (OUT_INJ3_(PD11))
- net INJ4: now also M4.E14 (OUT_INJ4_(PD10))
- net IN_AV_107: now also M4.S16 (IN_CAM_(PA6))
- net IN_AV_109: now also M4.S12 (IN_MAP2_(PC1))
- net IN_AV_110: now also M4.S9 (IN_AUX1_(PB0))
- net IN_AV_111: now also M4.S8 (IN_AUX2_(PC4/PE9))
- net IN_AV_112: now also M4.S7 (IN_AUX3_(PC5))
- net IN_AV_119: now also M4.S6 (IN_AUX4_(PA7))
- net IN_CAM: now also M4.S4 (IN_D1_(PE12))
- net IN_CLT: now also M4.S21 (IN_CLT_(PC2))
- net IN_DIGITAL_113: now also M4.S2 (IN_D3_(PE14))
- net IN_DIGITAL_120: now also M4.S1 (IN_D4_(PE15))
- net IN_IAT: now also M4.S20 (IN_IAT_(PC3))
- net IN_KNOCK: now also M4.S15 (IN_KNOCK_(PA2))
- net IN_MAP: now also M4.S13 (IN_MAP1_(PC0))
- net IN_PPS1: now also M4.S19 (IN_PPS_(PA3))
- net IN_PPS2: now also M4.S10 (IN_O2S2_(PA1))
- net IN_TPS1: now also M4.S18 (IN_TPS_(PA4))
- net IN_TPS2: now also M4.S11 (IN_O2S_/_CAN_WAKEUP_(PA0))
- net IN_VSS: now also M4.S3 (IN_D2_(PE13))
- net LS_101: now also M4.E13 (OUT_INJ5_(PD2))
- net LS_102: now also M4.E12 (OUT_INJ6_(PA8))
- net LS_235: now also M4.E11 (OUT_INJ7_(PD15))
- net LS_246: now also M4.E10 (OUT_INJ8_(PD12))
- net MAF_DIGITAL: now also M4.S17 (IN_VSS_(PE11))
- net MAIN_RELAY: now also M4.W3 (IGN8_(PE6))
- net PWR_EN: now also M4.N20 (OUT_PWR_EN_(PE10))
- net RELAY_140: now also M4.W4 (IGN7_(PB9))
- net RELAY_151: now also M4.W6 (IGN5_(PE2))
- net RELAY_152: now also M4.W5 (IGN6_(PB8))
- net TACH: now also M4.E18 (OUT_PWM1_(PD13))
- net TLS115_PG: now also M4.N9 (SPI3_CS_(PA15))
- net USB+: now also M4.N3 (USBP_(PA12))
- net USB-: now also M4.N2 (USBM_(PA11))
- net VBAT: now also M4.N17 (VBAT)
- net VBUS: now also M4.N1 (VBUS)
- net VIGN: now also M4.E5 (IN_VIGN_(PA5))
- net VREF2: now also M4.S5 (VREF2)
- net at M5.V2 (UART_RX), R92.2: now also M4.N18 (UART8_RX_(PE0))
- net at M5.V5 (UART_TX): now also M4.N19 (UART8_TX_(PE1))
- no-connect marks 54 -> 56
Other:
- moved on the sheet: J1
